Commit message: UAS

File: src/nav2_mobile_robot/urdf/gazebo_control.xacro (robot description, xacro)
@@ -14,5 +14,5 @@
       <publish_odom_tf>true</publish_odom_tf>
       <odom_publish_frequency>10</odom_publish_frequency>
-      <topic>cmd_vel</topic>
+      <topic>/cmd_vel</topic>
       <robotBaseFrame>base_link</robotBaseFrame>
     </plugin>

File: src/nav2_mobile_robot/urdf/lidar.xacro (robot description, xacro)
@@ -2,8 +2,8 @@
 <robot name="nav_robot"
   xmlns:xacro="http://ros.org/wiki/xacro">
-  <xacro:property name="PI" value="3.14159"/>
+  <xacro:property name="PI" value="3.14159" />
   <link name="lidar_link">
     <visual>
-      <origin xyz="0 0 0.05" rpy="0 0 0"/>
+      <origin xyz="0 0 0.05" rpy="0 0 0" />
       <geometry>
         <box size="0.05 0.05 0.05" />
@@ -11,5 +11,5 @@
     </visual>
     <collision>
-      <origin xyz="0 0 0.05" rpy="0 0 0"/>
+      <origin xyz="0 0 0.05" rpy="0 0 0" />
       <geometry>
         <box size="0.05 0.05 0.05" />
@@ -17,12 +17,12 @@
     </collision>
     <inertial>
-      <origin xyz="0 0 0.05" rpy="0 0 0"/>
-      <mass value="1"/>
-      <inertia ixx="1.0" ixy="0.0" ixz="0.0" iyy="1.0" iyz="0.0" izz="1.0"/>
+      <origin xyz="0 0 0.05" rpy="0 0 0" />
+      <mass value="1" />
+      <inertia ixx="1.0" ixy="0.0" ixz="0.0" iyy="1.0" iyz="0.0" izz="1.0" />
     </inertial>
   </link>
   <joint name='lidar_sensor_joint' type='fixed'>
-    <parent link="base_link"/>
-    <child link="lidar_link"/>
+    <parent link="base_link" />
+    <child link="lidar_link" />
   </joint>
   <gazebo reference="lidar_link">
@@ -36,9 +36,10 @@
             <samples>640</samples>
             <resolution>1</resolution>
-            <min_angle>-1.396263</min_angle>
-            <max_angle>1.396263</max_angle>
+            <!-- -pi sampai +pi = 360 derajat -->
+            <min_angle>-3.141593</min_angle>
+            <max_angle>3.141593</max_angle>
           </horizontal>
           <vertical>
-            <samples>16</samples>
+            <samples>36</samples>
             <resolution>1</resolution>
             <min_angle>-0.261799</min_angle>
@@ -47,5 +48,4 @@
         </scan>
         <range>
-          <!-- <min>0.08</min> -->
           <min>0.1</min>
           <max>10.0</max>

File: src/nav2_mobile_robot/urdf/nav2_mobile_robot_macro.xacro (robot description, xacro)
@@ -8,4 +8,7 @@
   <material name="White">
     <color rgba="1 1 1 1" />
+  </material>
+  <material name="Red">
+    <color rgba="1 0 0 0" />
   </material>
   <xacro:macro name="cylinder_inertia" params="m r h">
